File: AB Duplo diferencial.sch (KiCad schematic (older format))
At the start: 44 parts, among them Q1 C945, Q10 13007, Q11 13007, Q2 C945, Q3 A733, Q4 A733, Q5 A733, Q6 13003, Q7 C945, Q8 TIP41, Q9 TIP42

Commit message: Otimizadas algumas trilhas & adicionado resistor 4.7k da entrada pro terra para reduzir o ruído de 60hz
Parts:
- removed R16: 100R, Resistor_THT:R_Axial_DIN0204_L3.6mm_D1.6mm_P7.62mm_Horizontal, symbol Device:R
- C1: footprint Capacitor_THT:CP_Radial_D4.0mm_P1.50mm -> Capacitor_THT:CP_Radial_D5.0mm_P2.50mm
- R12, R13: value 10r -> 1k; footprint Resistor_THT:R_Axial_DIN0204_L3.6mm_D1.6mm_P7.62mm_Horizontal -> Resistor_THT:R_Axial_DIN0207_L6.3mm_D2.5mm_P10.16mm_Horizontal
- R15: value 100R -> 4,7k
Connections:
- wire segments 109 -> 104
Changed lines of the file:
@@
 F 0 "C1" V 1575 2000 50  0000 C CNN
 F 1 "2.2uf" V 1666 2000 50  0000 C CNN
-F 2 "Capacitor_THT:CP_Radial_D4.0mm_P1.50mm" H 1800 2000 50  0001 C CNN
+F 2 "Capacitor_THT:CP_Radial_D5.0mm_P2.50mm" H 1800 2000 50  0001 C CNN
 F 3 "" H 1800 2000 50  0001 C CNN
 	1    1800 2000
@@
 L Device:R R1
 U 1 1 6091F8B6
-P 1500 2000
-F 0 "R1" V 1293 2000 50  0000 C CNN
-F 1 "2k" V 1384 2000 50  0000 C CNN
-F 2 "Resistor_THT:R_Axial_DIN0204_L3.6mm_D1.6mm_P7.62mm_Horizontal" V 1430 2000 50  0001 C CNN
-F 3 "" H 1500 2000 50  0001 C CNN
-	1    1500 2000
+P 1450 2000
+F 0 "R1" V 1243 2000 50  0000 C CNN
+F 1 "2k" V 1334 2000 50  0000 C CNN
+F 2 "Resistor_THT:R_Axial_DIN0204_L3.6mm_D1.6mm_P7.62mm_Horizontal" V 1380 2000 50  0001 C CNN
+F 3 "" H 1450 2000 50  0001 C CNN
+	1    1450 2000
 	0    1    1    0
 $EndComp
@@
 	1    0    0    -1
 $EndComp
-Wire Wire Line
-	5200 3900 5600 3900
 $Comp
 L Connector:Conn_01x01_Male Sinal(+)1
 U 1 1 608B68B8
-P 1200 2000
-F 0 "Sinal(+)1" H 1306 2178 50  0000 C CNN
-F 1 "Sinal(+)" H 1306 2087 50  0000 C CNN
-F 2 "Connector_Wire:SolderWirePad_1x01_Drill0.8mm" H 1200 2000 50  0001 C CNN
-F 3 "~" H 1200 2000 50  0001 C CNN
-	1    1200 2000
-	1    0    0    -1
-$EndComp
-Wire Wire Line
-	1650 2000 1700 2000
+P 1100 2000
+F 0 "Sinal(+)1" H 1206 2178 50  0000 C CNN
+F 1 "Sinal(+)" H 1206 2087 50  0000 C CNN
+F 2 "Connector_Wire:SolderWirePad_1x01_Drill0.8mm" H 1100 2000 50  0001 C CNN
+F 3 "~" H 1100 2000 50  0001 C CNN
+	1    1100 2000
+	1    0    0    -1
+$EndComp
 $Comp
 L Connector:Conn_01x01_Male SAÍDA1
@@
 $EndComp
 Wire Wire Line
-	1350 2000 1400 2000
-Wire Wire Line
 	4400 3900 4400 3750
 $Comp
@@
 Connection ~ 2000 2000
 Wire Wire Line
-	3500 2900 2500 2900
-Wire Wire Line
 	2500 2900 2500 2000
 Connection ~ 2500 2000
@@
 P 5200 1100
 F 0 "R12" H 5130 1054 50  0000 R CNN
-F 1 "10r" H 5130 1145 50  0000 R CNN
-F 2 "Resistor_THT:R_Axial_DIN0204_L3.6mm_D1.6mm_P7.62mm_Horizontal" V 5130 1100 50  0001 C CNN
+F 1 "1k" H 5130 1145 50  0000 R CNN
+F 2 "Resistor_THT:R_Axial_DIN0207_L6.3mm_D2.5mm_P10.16mm_Horizontal" V 5130 1100 50  0001 C CNN
 F 3 "" H 5200 1100 50  0001 C CNN
 	1    5200 1100
@@
 P 5200 3600
 F 0 "R13" H 5130 3554 50  0000 R CNN
-F 1 "10r" H 5130 3645 50  0000 R CNN
-F 2 "Resistor_THT:R_Axial_DIN0204_L3.6mm_D1.6mm_P7.62mm_Horizontal" V 5130 3600 50  0001 C CNN
+F 1 "1k" H 5130 3645 50  0000 R CNN
+F 2 "Resistor_THT:R_Axial_DIN0207_L6.3mm_D2.5mm_P10.16mm_Horizontal" V 5130 3600 50  0001 C CNN
 F 3 "" H 5200 3600 50  0001 C CNN
 	1    5200 3600
@@
 	2200 2000 2200 2150
 Connection ~ 2200 2000
-Wire Wire Line
-	2200 2000 2500 2000
 $Comp
 L power:Earth #PWR02
@@
 	1    0    0    -1
 $EndComp
-Wire Wire Line
-	6600 3600 6600 3250
-Wire Wire Line
-	6600 3250 6900 3250
 $Comp
 L Device:R R20
@@
 Wire Wire Line
 	2000 4000 8050 4000
+Wire Wire Line
+	2200 2600 3350 2600
+Wire Wire Line
+	2000 4000 2000 2600
+Wire Wire Line
+	6300 900  6700 900
+Wire Wire Line
+	6300 3900 6750 3900
+Wire Wire Line
+	5200 3900 6300 3900
+Wire Wire Line
+	1600 2000 1700 2000
 $Comp
 L Device:R R15
-U 1 1 609DF472
-P 5600 2050
-F 0 "R15" H 5670 2096 50  0000 L CNN
-F 1 "100R" H 5670 2005 50  0000 L CNN
-F 2 "Resistor_THT:R_Axial_DIN0204_L3.6mm_D1.6mm_P7.62mm_Horizontal" V 5530 2050 50  0001 C CNN
-F 3 "~" H 5600 2050 50  0001 C CNN
-	1    5600 2050
-	1    0    0    -1
-$EndComp
-$Comp
-L Device:R R16
-U 1 1 609DF620
-P 5600 3500
-F 0 "R16" H 5670 3546 50  0000 L CNN
-F 1 "100R" H 5670 3455 50  0000 L CNN
-F 2 "Resistor_THT:R_Axial_DIN0204_L3.6mm_D1.6mm_P7.62mm_Horizontal" V 5530 3500 50  0001 C CNN
-F 3 "~" H 5600 3500 50  0001 C CNN
-	1    5600 3500
-	1    0    0    -1
-$EndComp
-Wire Wire Line
-	5600 3650 5600 3900
-Connection ~ 5600 3900
-Wire Wire Line
-	5600 3900 6300 3900
-Wire Wire Line
-	5600 3350 5600 3100
-Connection ~ 5600 3100
-Wire Wire Line
-	5600 2200 5600 2400
-Wire Wire Line
-	5600 1900 5600 1800
-Connection ~ 5600 1800
-Wire Wire Line
-	2200 2600 3350 2600
-Wire Wire Line
-	2000 4000 2000 2600
-Wire Wire Line
-	6300 900  6700 900
-Wire Wire Line
-	6300 3900 6750 3900
+U 1 1 63F30873
+P 1300 2300
+F 0 "R15" H 1230 2254 50  0000 R CNN
+F 1 "4,7k" H 1230 2345 50  0000 R CNN
+F 2 "Resistor_THT:R_Axial_DIN0204_L3.6mm_D1.6mm_P7.62mm_Horizontal" V 1230 2300 50  0001 C CNN
+F 3 "" H 1300 2300 50  0001 C CNN
+	1    1300 2300
+	-1   0    0    1
+$EndComp
+Wire Wire Line
+	2000 2600 1300 2600
+Wire Wire Line
+	1300 2600 1300 2450
+Wire Wire Line
+	1300 2150 1300 2000
+Connection ~ 1300 2000
+Wire Wire Line
+	2500 2900 3500 2900
+Wire Wire Line
+	2200 2000 2500 2000
 $EndSCHEMATC

Commit message: Alteradas rotas para R7 e R11 & expandido placa geral 1 furo para esquerda
Parts:
- removed R20: 10r, Resistor_THT:R_Axial_DIN0207_L6.3mm_D2.5mm_P10.16mm_Horizontal, symbol Device:R
- added R16: 10r, Resistor_THT:R_Axial_DIN0207_L6.3mm_D2.5mm_P10.16mm_Horizontal, symbol Device:R
Connections:
- wire segments 104 -> 105
Changed lines of the file:
@@
 	1    0    0    -1
-$EndComp
-$Comp
-L Device:R R20
-U 1 1 60963EEC
-P 7250 2500
-F 0 "R20" V 7043 2500 50  0000 C CNN
-F 1 "10r" V 7134 2500 50  0000 C CNN
-F 2 "Resistor_THT:R_Axial_DIN0207_L6.3mm_D2.5mm_P10.16mm_Horizontal" V 7180 2500 50  0001 C CNN
-F 3 "" H 7250 2500 50  0001 C CNN
-	1    7250 2500
-	0    1    -1   0
 $EndComp
 Wire Wire Line
@@
 Wire Wire Line
 	5600 2400 6300 2400
-$Comp
-L Device:L_Small L1
-U 1 1 609BF0F1
-P 7250 2400
-F 0 "L1" H 7297 2446 50  0000 L CNN
-F 1 "L_Small" H 7297 2355 50  0000 L CNN
-F 2 "Inductor_THT:L_Axial_L5.3mm_D2.2mm_P10.16mm_Horizontal_Vishay_IM-1" H 7250 2400 50  0001 C CNN
-F 3 "~" H 7250 2400 50  0001 C CNN
-	1    7250 2400
-	0    -1   -1   0
-$EndComp
-Wire Wire Line
-	7350 2400 7400 2400
-Wire Wire Line
-	7400 2400 7400 2500
 Wire Wire Line
 	6900 2400 6900 2650
-Wire Wire Line
-	7100 2400 7100 2500
-Wire Wire Line
-	7150 2400 7100 2400
-Connection ~ 6900 2400
-Connection ~ 7100 2400
-Wire Wire Line
-	7100 2400 6900 2400
-Connection ~ 7400 2400
-Wire Wire Line
-	7400 2400 7650 2400
 Wire Wire Line
 	6900 3250 8050 3250
@@
 Wire Wire Line
 	2200 2000 2500 2000
+Wire Wire Line
+	6900 2400 7650 2400
+Connection ~ 6900 2400
+Wire Wire Line
+	8350 2000 8600 2000
+Wire Wire Line
+	8350 2000 8350 2100
+Connection ~ 8350 2000
+Wire Wire Line
+	8300 2000 8350 2000
+Wire Wire Line
+	8050 2000 7850 2000
+Wire Wire Line
+	8050 2000 8050 2100
+Connection ~ 8050 2000
+Wire Wire Line
+	8100 2000 8050 2000
+$Comp
+L Device:L_Small L1
+U 1 1 65D2AEB4
+P 8200 2000
+F 0 "L1" H 8247 2046 50  0000 L CNN
+F 1 "L_Small" H 8247 1955 50  0000 L CNN
+F 2 "Inductor_THT:L_Axial_L5.3mm_D2.2mm_P10.16mm_Horizontal_Vishay_IM-1" H 8200 2000 50  0001 C CNN
+F 3 "~" H 8200 2000 50  0001 C CNN
+	1    8200 2000
+	0    -1   -1   0
+$EndComp
+$Comp
+L Device:R R16
+U 1 1 65D2AEBB
+P 8200 2100
+F 0 "R16" V 7993 2100 50  0000 C CNN
+F 1 "10r" V 8084 2100 50  0000 C CNN
+F 2 "Resistor_THT:R_Axial_DIN0207_L6.3mm_D2.5mm_P10.16mm_Horizontal" V 8130 2100 50  0001 C CNN
+F 3 "" H 8200 2100 50  0001 C CNN
+	1    8200 2100
+	0    1    -1   0
+$EndComp
 $EndSCHEMATC

Commit message: [atualizados] Valores: C7(47uf) & R2/R14(100k) & R12/R13(2K) & R15(10K) [renomeados] "Sinal(+)" para "P2" & +VCC1 para "+24" & "-VCC1" para "-24" & "SAÍDA" para "Falante"
Parts:
- removed L1: L_Small, Inductor_THT:L_Axial_L5.3mm_D2.2mm_P10.16mm_Horizontal_Vishay_IM-1, symbol Device:L_Small
- removed R16: 10r, Resistor_THT:R_Axial_DIN0207_L6.3mm_D2.5mm_P10.16mm_Horizontal, symbol Device:R
- +VCC1: value +VCC -> +24
- -VCC1: value -VCC -> -24
- C3: value 100uf -> 47uf
- C4, C5: value 47pf -> 100pf
- Q6: value 13003 -> C945
- R12, R13: value 1k -> 2k
- R14, R2: value 47k -> 100k
- R15: value 4,7k -> 10k
- SAÍDA1: value SAÍDA -> Falante
- Sinal(+)1: value Sinal(+) -> P2(+)
Connections:
- wire segments 105 -> 99
Changed lines of the file:
@@
 P 5000 2900
 F 0 "C5" V 4771 2900 50  0000 C CNN
-F 1 "47pf" V 4862 2900 50  0000 C CNN
+F 1 "100pf" V 4862 2900 50  0000 C CNN
 F 2 "Capacitor_THT:C_Disc_D3.0mm_W1.6mm_P2.50mm" H 5000 2900 50  0001 C CNN
 F 3 "" H 5000 2900 50  0001 C CNN
@@
 P 5400 2400
 F 0 "R14" V 5193 2400 50  0000 C CNN
-F 1 "47k" V 5284 2400 50  0000 C CNN
+F 1 "100k" V 5284 2400 50  0000 C CNN
 F 2 "Resistor_THT:R_Axial_DIN0204_L3.6mm_D1.6mm_P7.62mm_Horizontal" V 5330 2400 50  0001 C CNN
 F 3 "" H 5400 2400 50  0001 C CNN
@@
 P 3900 2200
 F 0 "C3" H 3988 2246 50  0000 L CNN
-F 1 "100uf" H 3988 2155 50  0000 L CNN
+F 1 "47uf" H 3988 2155 50  0000 L CNN
 F 2 "Capacitor_THT:CP_Radial_D7.5mm_P2.50mm" H 3900 2200 50  0001 C CNN
 F 3 "" H 3900 2200 50  0001 C CNN
@@
 P 2200 2300
 F 0 "R2" H 2130 2254 50  0000 R CNN
-F 1 "47k" H 2130 2345 50  0000 R CNN
+F 1 "100k" H 2130 2345 50  0000 R CNN
 F 2 "Resistor_THT:R_Axial_DIN0204_L3.6mm_D1.6mm_P7.62mm_Horizontal" V 2130 2300 50  0001 C CNN
 F 3 "" H 2200 2300 50  0001 C CNN
@@
 P 6950 3900
 F 0 "-VCC1" H 6977 3926 50  0000 L CNN
-F 1 "-VCC" H 6977 3835 50  0000 L CNN
+F 1 "-24" H 6977 3835 50  0000 L CNN
 F 2 "Connector_Wire:SolderWirePad_1x01_Drill0.8mm" H 6950 3900 50  0001 C CNN
 F 3 "~" H 6950 3900 50  0001 C CNN
@@
 P 6900 900
 F 0 "+VCC1" H 6927 926 50  0000 L CNN
-F 1 "+VCC" H 6927 835 50  0000 L CNN
+F 1 "+24" H 6927 835 50  0000 L CNN
 F 2 "Connector_Wire:SolderWirePad_1x01_Drill0.8mm" H 6900 900 50  0001 C CNN
 F 3 "~" H 6900 900 50  0001 C CNN
@@
 P 1100 2000
 F 0 "Sinal(+)1" H 1206 2178 50  0000 C CNN
-F 1 "Sinal(+)" H 1206 2087 50  0000 C CNN
+F 1 "P2(+)" H 1206 2087 50  0000 C CNN
 F 2 "Connector_Wire:SolderWirePad_1x01_Drill0.8mm" H 1100 2000 50  0001 C CNN
 F 3 "~" H 1100 2000 50  0001 C CNN
@@
 P 7850 2400
 F 0 "SAÍDA1" V 7910 2312 50  0000 R CNN
-F 1 "SAÍDA" V 8001 2312 50  0000 R CNN
+F 1 "Falante" V 8001 2312 50  0000 R CNN
 F 2 "Connector_Wire:SolderWirePad_1x01_Drill0.8mm" H 7850 2400 50  0001 C CNN
 F 3 "~" H 7850 2400 50  0001 C CNN
@@
 P 5200 1100
 F 0 "R12" H 5130 1054 50  0000 R CNN
-F 1 "1k" H 5130 1145 50  0000 R CNN
+F 1 "2k" H 5130 1145 50  0000 R CNN
 F 2 "Resistor_THT:R_Axial_DIN0207_L6.3mm_D2.5mm_P10.16mm_Horizontal" V 5130 1100 50  0001 C CNN
 F 3 "" H 5200 1100 50  0001 C CNN
@@
 P 5200 3600
 F 0 "R13" H 5130 3554 50  0000 R CNN
-F 1 "1k" H 5130 3645 50  0000 R CNN
+F 1 "2k" H 5130 3645 50  0000 R CNN
 F 2 "Resistor_THT:R_Axial_DIN0207_L6.3mm_D2.5mm_P10.16mm_Horizontal" V 5130 3600 50  0001 C CNN
 F 3 "" H 5200 3600 50  0001 C CNN
@@
 P 5000 1600
 F 0 "C4" V 4771 1600 50  0000 C CNN
-F 1 "47pf" V 4862 1600 50  0000 C CNN
+F 1 "100pf" V 4862 1600 50  0000 C CNN
 F 2 "Capacitor_THT:C_Disc_D3.0mm_W1.6mm_P2.50mm" H 5000 1600 50  0001 C CNN
 F 3 "" H 5000 1600 50  0001 C CNN
@@
 P 5100 2000
 F 0 "Q6" H 5291 2046 50  0000 L CNN
-F 1 "13003" H 5291 1955 50  0000 L CNN
+F 1 "C945" H 5291 1955 50  0000 L CNN
 F 2 "Package_TO_SOT_THT:TO-126-3_Vertical" H 5300 2100 50  0001 C CNN
 F 3 "~" H 5100 2000 50  0001 C CNN
@@
 P 1300 2300
 F 0 "R15" H 1230 2254 50  0000 R CNN
-F 1 "4,7k" H 1230 2345 50  0000 R CNN
+F 1 "10k" H 1230 2345 50  0000 R CNN
 F 2 "Resistor_THT:R_Axial_DIN0204_L3.6mm_D1.6mm_P7.62mm_Horizontal" V 1230 2300 50  0001 C CNN
 F 3 "" H 1300 2300 50  0001 C CNN
@@
 	6900 2400 7650 2400
 Connection ~ 6900 2400
-Wire Wire Line
-	8350 2000 8600 2000
-Wire Wire Line
-	8350 2000 8350 2100
-Connection ~ 8350 2000
-Wire Wire Line
-	8300 2000 8350 2000
-Wire Wire Line
-	8050 2000 7850 2000
-Wire Wire Line
-	8050 2000 8050 2100
-Connection ~ 8050 2000
-Wire Wire Line
-	8100 2000 8050 2000
-$Comp
-L Device:L_Small L1
-U 1 1 65D2AEB4
-P 8200 2000
-F 0 "L1" H 8247 2046 50  0000 L CNN
-F 1 "L_Small" H 8247 1955 50  0000 L CNN
-F 2 "Inductor_THT:L_Axial_L5.3mm_D2.2mm_P10.16mm_Horizontal_Vishay_IM-1" H 8200 2000 50  0001 C CNN
-F 3 "~" H 8200 2000 50  0001 C CNN
-	1    8200 2000
-	0    -1   -1   0
-$EndComp
-$Comp
-L Device:R R16
-U 1 1 65D2AEBB
-P 8200 2100
-F 0 "R16" V 7993 2100 50  0000 C CNN
-F 1 "10r" V 8084 2100 50  0000 C CNN
-F 2 "Resistor_THT:R_Axial_DIN0207_L6.3mm_D2.5mm_P10.16mm_Horizontal" V 8130 2100 50  0001 C CNN
-F 3 "" H 8200 2100 50  0001 C CNN
-	1    8200 2100
-	0    1    -1   0
-$EndComp
 $EndSCHEMATC

Commit message: [rollback] R2 & R14 pra 47k [alterado] C4 & C5 pra 47pf
Parts:
- C4, C5: value 100pf -> 47pf
- R14, R2: value 100k -> 47k
Changed lines of the file:
@@
 P 5000 2900
 F 0 "C5" V 4771 2900 50  0000 C CNN
-F 1 "100pf" V 4862 2900 50  0000 C CNN
+F 1 "47pf" V 4862 2900 50  0000 C CNN
 F 2 "Capacitor_THT:C_Disc_D3.0mm_W1.6mm_P2.50mm" H 5000 2900 50  0001 C CNN
 F 3 "" H 5000 2900 50  0001 C CNN
@@
 P 5400 2400
 F 0 "R14" V 5193 2400 50  0000 C CNN
-F 1 "100k" V 5284 2400 50  0000 C CNN
+F 1 "47k" V 5284 2400 50  0000 C CNN
 F 2 "Resistor_THT:R_Axial_DIN0204_L3.6mm_D1.6mm_P7.62mm_Horizontal" V 5330 2400 50  0001 C CNN
 F 3 "" H 5400 2400 50  0001 C CNN
@@
 P 2200 2300
 F 0 "R2" H 2130 2254 50  0000 R CNN
-F 1 "100k" H 2130 2345 50  0000 R CNN
+F 1 "47k" H 2130 2345 50  0000 R CNN
 F 2 "Resistor_THT:R_Axial_DIN0204_L3.6mm_D1.6mm_P7.62mm_Horizontal" V 2130 2300 50  0001 C CNN
 F 3 "" H 2200 2300 50  0001 C CNN
@@
 P 5000 1600
 F 0 "C4" V 4771 1600 50  0000 C CNN
-F 1 "100pf" V 4862 1600 50  0000 C CNN
+F 1 "47pf" V 4862 1600 50  0000 C CNN
 F 2 "Capacitor_THT:C_Disc_D3.0mm_W1.6mm_P2.50mm" H 5000 1600 50  0001 C CNN
 F 3 "" H 5000 1600 50  0001 C CNN

Commit message: [corrigido] TO-92_Inline pra TO-92_Inline_Wide & visão 3d no PcbView
Parts:
- Q1, Q2, Q3, Q4, Q5, Q7: footprint Package_TO_SOT_THT:TO-92_Inline -> Package_TO_SOT_THT:TO-92_Inline_Wide
Changed lines of the file:
@@
 F 0 "Q7" H 5291 3246 50  0000 L CNN
 F 1 "C945" H 5291 3155 50  0000 L CNN
-F 2 "Package_TO_SOT_THT:TO-92_Inline" H 5300 3300 50  0001 C CNN
+F 2 "Package_TO_SOT_THT:TO-92_Inline_Wide" H 5300 3300 50  0001 C CNN
 F 3 "" H 5100 3200 50  0001 C CNN
 	1    5100 3200
@@
 F 0 "Q4" H 4691 2854 50  0000 L CNN
 F 1 "A733" H 4691 2945 50  0000 L CNN
-F 2 "Package_TO_SOT_THT:TO-92_Inline" H 4700 3000 50  0001 C CNN
+F 2 "Package_TO_SOT_THT:TO-92_Inline_Wide" H 4700 3000 50  0001 C CNN
 F 3 "" H 4500 2900 50  0001 C CNN
 	1    4500 2900
@@
 F 0 "Q3" H 3891 2854 50  0000 L CNN
 F 1 "A733" H 3891 2945 50  0000 L CNN
-F 2 "Package_TO_SOT_THT:TO-92_Inline" H 3900 3000 50  0001 C CNN
+F 2 "Package_TO_SOT_THT:TO-92_Inline_Wide" H 3900 3000 50  0001 C CNN
 F 3 "" H 3700 2900 50  0001 C CNN
 	1    3700 2900
@@
 F 0 "Q2" H 3690 2046 50  0000 L CNN
 F 1 "C945" H 3690 1955 50  0000 L CNN
-F 2 "Package_TO_SOT_THT:TO-92_Inline" H 3700 2100 50  0001 C CNN
+F 2 "Package_TO_SOT_THT:TO-92_Inline_Wide" H 3700 2100 50  0001 C CNN
 F 3 "~" H 3500 2000 50  0001 C CNN
 	1    3500 2000
@@
 F 0 "Q1" H 2891 2046 50  0000 L CNN
 F 1 "C945" H 2891 1955 50  0000 L CNN
-F 2 "Package_TO_SOT_THT:TO-92_Inline" H 2900 2100 50  0001 C CNN
+F 2 "Package_TO_SOT_THT:TO-92_Inline_Wide" H 2900 2100 50  0001 C CNN
 F 3 "~" H 2700 2000 50  0001 C CNN
 	1    2700 2000
@@
 F 0 "Q5" H 5291 1354 50  0000 L CNN
 F 1 "A733" H 5291 1445 50  0000 L CNN
-F 2 "Package_TO_SOT_THT:TO-92_Inline" H 5300 1500 50  0001 C CNN
+F 2 "Package_TO_SOT_THT:TO-92_Inline_Wide" H 5300 1500 50  0001 C CNN
 F 3 "" H 5100 1400 50  0001 C CNN
 	1    5100 1400
